Commit message: Add chassis

File: diff-drive-robot-description/description/robot.urdf.xacro (robot description, xacro)
@@ -3,3 +3,18 @@
 	<link name="base_link">
 	</link>
+	<!-- Chassis Link -->
+	<joint name="chassis_joint" type="fixed">
+		<parent link="base_link"/>
+		<child link="chassis"/>
+		<origin xyz="-0.1 0 0 "/>
+	</joint>
+	<link name="chassis">
+		<visual>
+			<origin xyz="0.15 0 0.075"/>
+			 <geometry>
+				 <box size="o.3 0.03 0.15"/>
+			</geometry>
+			<material name="white"/>
+		</visual>
+	</link>
 </robot>

Commit message: Fix chassis errors

File: diff-drive-robot-description/description/robot.urdf.xacro (robot description, xacro)
@@ -1,4 +1,7 @@
 <?xml version="1.0"?>
 <robot xmlns:xacro="http://www.ros.org/wiki/xacro" name="robot">
+	<material name="white">
+		<color rgba="1 1 1 1"/>
+	</material>
 	<link name="base_link">
 	</link>
@@ -13,5 +16,5 @@
 			<origin xyz="0.15 0 0.075"/>
 			 <geometry>
-				 <box size="o.3 0.03 0.15"/>
+				 <box size="0.3 0.3 0.15"/>
 			</geometry>
 			<material name="white"/>

Commit message: Add wheels

File: diff-drive-robot-description/description/robot.urdf.xacro (robot description, xacro)
@@ -4,7 +4,11 @@
 		<color rgba="1 1 1 1"/>
 	</material>
+	<material name="blue">
+		<color rgba="0.2 0.2 1 1"/>
+	</material>
+	<!-- Base link -->
 	<link name="base_link">
 	</link>
-	<!-- Chassis Link -->
+	<!-- Chassis -->
 	<joint name="chassis_joint" type="fixed">
 		<parent link="base_link"/>
@@ -21,3 +25,33 @@
 		</visual>
 	</link>
+	<!-- Left Wheel -->
+	<joint name="left_wheel_joint" type="continuous">
+		<parent link="base_link"/>
+		<child link="left_wheel"/>
+		<origin xyz="0 0.175 0" rpy="-${pi/2} 0 0" />
+		<axis xyz="0 0 1"/>
+	</joint>
+	<link name="left_wheel">
+		<visual>
+			<geometry>
+				<cylinder radius="0.05" length="0.04"/>
+			</geometry>
+			<material name="blue"/>
+		</visual>
+	</link>
+	<!-- Right Wheel -->
+	<joint name="right_wheel_joint" type="continuous">
+		<parent link="base_link"/>
+		<child link="right_wheel"/>
+		<origin xyz="0 -0.175 0" rpy="${pi/2} 0 0" />
+		<axis xyz="0 0 -1"/>
+	</joint>
+	<link name="right_wheel">
+		<visual>
+			<geometry>
+				<cylinder radius="0.05" length="0.04"/>
+			</geometry>
+			<material name="blue"/>
+		</visual>
+	</link>
 </robot>

Commit message: Add caster wheel

File: diff-drive-robot-description/description/robot.urdf.xacro (robot description, xacro)
@@ -55,3 +55,17 @@
 		</visual>
 	</link>
+	<!-- Caster wheel -->
+	<joint name="caster_wheel_joint" type="fixed">
+		<parent link="chassis"/>
+		<child link="caster_wheel"/>
+		<origin xyz="0.24 0 0"/>
+	</joint>
+	<link name="caster_wheel">
+		<visual>
+			<geometry>
+				<sphere radius="0.05"/>
+			</geometry>
+			<material name="black"/>
+		</visual>
+	</link>
 </robot>
